Commit message: paolo: update master

File: tez_description/urdf/tez_cell_boxes.urdf (robot description, URDF)
Before this commit: robot tez_cell, 17 links, 16 joints
Links:
- link jig: geometry collision mesh filename=package://tez_description/mesh/reduced_details/jig.dae; visual mesh filename=package://tez_description/mesh/reduced_details/jig.dae
- link linear_axis: geometry collision mesh filename=package://tez_description/mesh/full_details/linear_axis.dae; visual mesh filename=package://tez_description/mesh/full_details/linear_axis.dae

File: tez_description/urdf/tez_cell_fullmesh.urdf (robot description, URDF)
Before this commit: robot tez_cell, 17 links, 16 joints
Links:
- removed link jig
- link KR210_1_A1: geometry collision mesh filename=package://tez_description/mesh/full_details/KR210_3100_ultr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; visual mesh filename=package://tez_description/mesh/full_details/KR210_3100_ultr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
- link KR210_1_A2: geometry collision mesh filename=package://tez_description/mesh/full_details/KR210_3100_ultr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; visual mesh filename=package://tez_description/mesh/full_details/KR210_3100_ultr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
- link KR210_1_A3: geometry collision mesh filename=package://tez_description/mesh/full_details/KR210_3100_ultr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; visual mesh filename=package://tez_description/mesh/full_details/KR210_3100_ultr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
- link KR210_1_A4: geometry collision mesh filename=package://tez_description/mesh/full_details/KR210_3100_ultr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; visual mesh filename=package://tez_description/mesh/full_details/KR210_3100_ultr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
- link KR210_1_A5: geometry collision mesh filename=package://tez_description/mesh/full_details/KR210_3100_ultr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; visual mesh filename=package://tez_description/mesh/full_details/KR210_3100_ultr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
- link KR210_1_A6: geometry collision mesh filename=package://tez_description/mesh/full_details/KR210_3100_ultr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; visual mesh filename=package://tez_description/mesh/full_details/KR210_3100_ultr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
- link KR210_1_socket: geometry collision mesh filename=package://tez_description/mesh/full_details/KR210_3100_ultr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; visual mesh filename=package://tez_description/mesh/full_details/KR210_3100_ultr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
- link KR210_2_A1: geometry collision mesh filename=package://tez_description/mesh/full_details/KR210_3100_ultr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; visual mesh filename=package://tez_description/mesh/full_details/KR210_3100_ultr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
- link KR210_2_A2: geometry collision mesh filename=package://tez_description/mesh/full_details/KR210_3100_ultr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; visual mesh filename=package://tez_description/mesh/full_details/KR210_3100_ultr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
- link KR210_2_A3: geometry collision mesh filename=package://tez_description/mesh/full_details/KR210_3100_ultr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; visual mesh filename=package://tez_description/mesh/full_details/KR210_3100_ultr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
- link KR210_2_A4: geometry collision mesh filename=package://tez_description/mesh/full_details/KR210_3100_ultr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; visual mesh filename=package://tez_description/mesh/full_details/KR210_3100_ultr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
- link KR210_2_A5: geometry collision mesh filename=package://tez_description/mesh/full_details/KR210_3100_ultr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; visual mesh filename=package://tez_description/mesh/full_details/KR210_3100_ultr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
- link KR210_2_A6: geometry collision mesh filename=package://tez_description/mesh/full_details/KR210_3100_ultr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; visual mesh filename=package://tez_description/mesh/full_details/KR210_3100_ultr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
- link KR210_2_socket: geometry collision mesh filename=package://tez_description/mesh/full_details/KR210_3100_ultr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; visual mesh filename=package://tez_description/mesh/full_details/KR210_3100_ultr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
- link base_link: geometry collision mesh filename=package://tez_description/mesh/full_details/spannfeld.dae; visual mesh filename=package://tez_description/mesh/full_details/spannfeld.dae
- link linear_axis: geometry collision mesh filename=package://tez_description/mesh/full_details/linear_axis.dae; visual mesh filename=package://tez_description/mesh/full_details/linear_axis.dae
Joints:
- removed joint jig_pos
- joint kr210_1_joint_1: axis 0.0 0.0 1.0 -> 0.0 0.0 -1.0; limit lower=-3.22886 upper=3.22886 effort=100 velocity=100 -> lower=-3.22886 upper=3.22886 effort=100 velocity=1; origin xyz=0 0 0.5256 rpy=0 0 0 -> xyz=0 0 0.5256 rpy=0 0 -1.5707963267948966
- joint kr210_1_joint_2: limit lower=-2.0944 upper=1.22173 effort=10000 velocity=100 -> lower=-2.443460952792061 upper=-0.08726646259971647 effort=10000 velocity=1; origin xyz=0.005 -0.35 0.45 rpy=0 0 0 -> xyz=0.005 -0.35 0.45 rpy=1.5707963267948966 0 0
- joint kr210_1_joint_3: limit lower=-2.0944 upper=2.70526 effort=100 velocity=100 -> lower=-2.0943951023931953 upper=2.705260340591211 effort=100 velocity=1; origin xyz=-0.183 0 1.35 rpy=0 0 0 -> xyz=-0.183 0 1.35 rpy=-1.5707963267948966 0 0
- joint kr210_1_joint_5: limit lower=-2.18166 upper=2.18166 effort=100 velocity=100 -> lower=-2.138028333693054 upper=2.138028333693054 effort=100 velocity=1
- joint kr210_1_linear_axis_joint: limit lower=0 upper=9 effort=100 velocity=100 -> lower=-9 upper=0 effort=100 velocity=100; origin xyz=0 0 0.487 rpy=0 0 3.14159 -> xyz=0 0 0.487 rpy=0 0 0

File: tez_description/urdf/tez_cell_reducedmesh.urdf (robot description, URDF)
Before this commit: robot tez_cell, 17 links, 16 joints
Links:
- removed link jig
- added link gripper; collision mesh filename=package://tez_description/mesh/collada/reduced_details/grip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; visual mesh filename=package://tez_description/mesh/collada/reduced_details/grip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
- link KR210_1_A1: geometry collision mesh filename=package://tez_description/mesh/reduced_details/KR210_3100_u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; visual mesh filename=package://tez_description/mesh/reduced_details/KR210_3100_u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
- link KR210_1_A2: geometry collision mesh filename=package://tez_description/mesh/reduced_details/KR210_3100_u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; visual mesh filename=package://tez_description/mesh/reduced_details/KR210_3100_u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
- link KR210_1_A3: geometry collision mesh filename=package://tez_description/mesh/reduced_details/KR210_3100_u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; visual mesh filename=package://tez_description/mesh/reduced_details/KR210_3100_u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
- link KR210_1_A4: geometry collision mesh filename=package://tez_description/mesh/reduced_details/KR210_3100_u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; visual mesh filename=package://tez_description/mesh/reduced_details/KR210_3100_u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
- link KR210_1_A5: geometry collision mesh filename=package://tez_description/mesh/reduced_details/KR210_3100_u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; visual mesh filename=package://tez_description/mesh/reduced_details/KR210_3100_u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
- link KR210_1_A6: geometry collision mesh filename=package://tez_description/mesh/reduced_details/KR210_3100_u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; visual mesh filename=package://tez_description/mesh/reduced_details/KR210_3100_u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
- link KR210_1_socket: geometry collision mesh filename=package://tez_description/mesh/reduced_details/KR210_3100_u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; visual mesh filename=package://tez_description/mesh/reduced_details/KR210_3100_u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
- link KR210_2_A1: geometry collision mesh filename=package://tez_description/mesh/reduced_details/KR210_3100_u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; visual mesh filename=package://tez_description/mesh/reduced_details/KR210_3100_u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
- link KR210_2_A2: geometry collision mesh filename=package://tez_description/mesh/reduced_details/KR210_3100_u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; visual mesh filename=package://tez_description/mesh/reduced_details/KR210_3100_u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
- link KR210_2_A3: geometry collision mesh filename=package://tez_description/mesh/reduced_details/KR210_3100_u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; visual mesh filename=package://tez_description/mesh/reduced_details/KR210_3100_u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
- link KR210_2_A4: geometry collision mesh filename=package://tez_description/mesh/reduced_details/KR210_3100_u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; visual mesh filename=package://tez_description/mesh/reduced_details/KR210_3100_u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
- link KR210_2_A5: geometry collision mesh filename=package://tez_description/mesh/reduced_details/KR210_3100_u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; visual mesh filename=package://tez_description/mesh/reduced_details/KR210_3100_u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
- link KR210_2_A6: geometry collision mesh filename=package://tez_description/mesh/reduced_details/KR210_3100_u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; visual mesh filename=package://tez_description/mesh/reduced_details/KR210_3100_u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
- link KR210_2_socket: geometry collision mesh filename=package://tez_description/mesh/reduced_details/KR210_3100_u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; visual mesh filename=package://tez_description/mesh/reduced_details/KR210_3100_u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
- link base_link: geometry collision mesh filename=package://tez_description/mesh/reduced_details/spannfeld.dae; visual mesh filename=package://tez_description/mesh/reduced_details/spannfeld.dae
- link linear_axis: geometry collision mesh filename=package://tez_description/mesh/reduced_details/linear_axis.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; visual mesh filename=package://tez_description/mesh/reduced_details/linear_axis.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
Joints:
- removed joint jig_pos
- added joint EndEffector: type fixed, parent KR210_2_A6, child gripper, origin xyz=0 -0.01 0 rpy=0 0 1.5708, axis 0 0 0
- joint kr210_1_joint_1: axis 0.0 0.0 1.0 -> 0.0 0.0 -1.0; limit lower=-3.22886 upper=3.22886 effort=100 velocity=100 -> lower=-3.22886 upper=3.22886 effort=100 velocity=0.1; origin xyz=0 0 0.5256 rpy=0 0 0 -> xyz=0 0 0.5256 rpy=0 0 -1.5707963267948966
- joint kr210_1_joint_2: limit lower=-2.0944 upper=1.22173 effort=10000 velocity=100 -> lower=-2.443460952792061 upper=-0.08726646259971647 effort=10000 velocity=0.1; origin xyz=0.005 -0.35 0.45 rpy=0 0 0 -> xyz=0.005 -0.35 0.45 rpy=1.5707963267948966 0 0
- joint kr210_1_joint_3: limit lower=-2.0944 upper=2.70526 effort=100 velocity=100 -> lower=-2.0943951023931953 upper=2.705260340591211 effort=100 velocity=0.1; origin xyz=-0.183 0 1.35 rpy=0 0 0 -> xyz=-0.183 0 1.35 rpy=-1.5707963267948966 0 0
- joint kr210_1_joint_5: limit lower=-2.18166 upper=2.18166 effort=100 velocity=100 -> lower=-2.138028333693054 upper=2.138028333693054 effort=100 velocity=0.1
- joint kr210_1_linear_axis_joint: limit lower=0 upper=9 effort=100 velocity=100 -> lower=-9 upper=0 effort=100 velocity=100; origin xyz=0 0 0.487 rpy=0 0 3.14159 -> xyz=0 0 0.487 rpy=0 0 0
- joint kr210_2_joint_1: axis 0.0 0.0 1.0 -> 0.0 0.0 -1.0; limit lower=-3.22886 upper=3.22886 effort=100 velocity=100 -> lower=-3.22886 upper=3.22886 effort=100 velocity=0.1; origin xyz=0 0 0.5256 rpy=0 0 0 -> xyz=0 0 0.5256 rpy=0 0 -1.5707963267948966
- joint kr210_2_joint_2: limit lower=-2.0944 upper=1.22173 effort=10000 velocity=100 -> lower=-2.443460952792061 upper=-0.08726646259971647 effort=10000 velocity=0.1; origin xyz=0.005 -0.35 0.45 rpy=0 0 0 -> xyz=0.005 -0.35 0.45 rpy=1.5707963267948966 0 0
- joint kr210_2_joint_3: limit lower=-2.0944 upper=2.70526 effort=100 velocity=100 -> lower=-2.0943951023931953 upper=2.705260340591211 effort=100 velocity=0.1; origin xyz=-0.183 0 1.35 rpy=0 0 0 -> xyz=-0.183 0 1.35 rpy=-1.5707963267948966 0 0
- joint kr210_2_joint_5: limit lower=-2.18166 upper=2.18166 effort=100 velocity=100 -> lower=-2.138028333693054 upper=2.138028333693054 effort=100 velocity=0.1
- joint kr210_2_linear_axis_joint: limit lower=1.5 upper=9 effort=100 velocity=100 -> lower=-9 upper=0 effort=100 velocity=100; origin xyz=-1.5 0 0.487 rpy=0 0 3.14159 -> xyz=-9.0 0 0.487 rpy=0 0 3.1415
